Commit message: velodyne

File: src/articubot_one/description/lidar.xacro (robot description, xacro)
@@ -1,4 +1,5 @@
 <?xml version="1.0"?>
 <robot xmlns:xacro="http://www.ros.org/wiki/xacro" >
+  <xacro:property name="M_PI" value="3.1415926535897931"/>
     <joint name="laser_joint" type="fixed">
         <parent link="chassis"/>
@@ -42,4 +43,10 @@
                         <max_angle>3.14</max_angle>
                     </horizontal>
+                    <vertical>
+                        <samples>360</samples>
+                        <resolution>1</resolution>
+                        <min_angle>-${15.0*M_PI/180.0}</min_angle>
+                        <max_angle>${15.0*M_PI/180.0}</max_angle>
+                    </vertical>
                 </scan>
                 <range>

Commit message: velodyne fix

File: src/articubot_one/description/lidar.xacro (robot description, xacro)
@@ -39,10 +39,11 @@
                 <scan>
                     <horizontal>
-                        <samples>360</samples>
+                        <samples>180</samples>
+                        <resolution>1</resolution>
                         <min_angle>-3.14</min_angle>
                         <max_angle>3.14</max_angle>
                     </horizontal>
                     <vertical>
-                        <samples>360</samples>
+                        <samples>16</samples>
                         <resolution>1</resolution>
                         <min_angle>-${15.0*M_PI/180.0}</min_angle>
@@ -54,11 +55,28 @@
                     <max>12</max>
                 </range>
+                <range>
+                    <min>0.3</min>
+                    <max>131.0</max>
+                    <resolution>0.001</resolution>
+                </range>
+                <noise>
+                    <type>gaussian</type>
+                    <mean>0.0</mean>
+                    <stddev>0.0</stddev>
+                </noise>
             </ray>
-            <plugin name="laser_controller" filename="libgazebo_ros_ray_sensor.so">
-                <ros>
-                    <argument>~/out:=scan</argument>
-                </ros>
-                <output_type>sensor_msgs/LaserScan</output_type>
-                <frame_name>laser_frame</frame_name>
+            <!-- <plugin name="gazebo_ros_laser_controller" filename="libgazebo_ros_velodyne_laser.so">
+                <topicName>/velodyne_points</topicName>
+                <frameName>velodyne</frameName>
+                <min_range>0.9</min_range>
+                <max_range>130.0</max_range>
+                <gaussianNoise>0.008</gaussianNoise>
+            </plugin> -->
+            <plugin name="laser_controller" filename="libgazebo_ros_velodyne_laser.so">
+                <topicName>/velodyne_points</topicName>
+                <frameName>laser_frame</frameName>
+                <min_range>0.9</min_range>
+                <max_range>130.0</max_range>
+                <gaussianNoise>0.008</gaussianNoise>
             </plugin>
         </sensor>

File: src/velodyne_description/urdf/HDL-32E.urdf.xacro (robot description, xacro)
@@ -2,5 +2,5 @@
 <robot xmlns:xacro="http://www.ros.org/wiki/xacro" name="HDL-32E">
   <xacro:property name="M_PI" value="3.1415926535897931" />
-  <xacro:macro name="HDL-32E" params="*origin parent:=base_link name:=velodyne topic:=/velodyne_points hz:=10 lasers:=32 samples:=2187 collision_range:=0.3 min_range:=0.9 max_range:=130.0 noise:=0.008 min_angle:=-${M_PI} max_angle:=${M_PI} gpu:=false">
+  <xacro:macro name="HDL-32E" params="*origin parent:=base_link name:=velodyne topic:=/velodyne_points hz:=10 lasers:=32 samples:=180 collision_range:=0.3 min_range:=0.9 max_range:=130.0 noise:=0.008 min_angle:=-${M_PI} max_angle:=${M_PI} gpu:=false">
     <joint name="${name}_base_mount_joint" type="fixed">
       <xacro:insert_block name="origin" />
@@ -51,5 +51,5 @@
         <sensor type="gpu_ray" name="${name}-HDL32E">
           <pose>0 0 0 0 0 0</pose>
-          <visualize>false</visualize>
+          <visualize>true</visualize>
           <update_rate>${hz}</update_rate>
           <ray>
@@ -91,5 +91,5 @@
         <sensor type="ray" name="${name}-HDL32E">
           <pose>0 0 0 0 0 0</pose>
-          <visualize>false</visualize>
+          <visualize>true</visualize>
           <update_rate>${hz}</update_rate>
           <ray>

File: src/velodyne_description/urdf/VLP-16.urdf.xacro (robot description, xacro)
@@ -54,5 +54,5 @@
         <sensor type="gpu_ray" name="${name}-VLP16">
           <pose>0 0 0 0 0 0</pose>
-          <visualize>false</visualize>
+          <visualize>true</visualize>
           <update_rate>${hz}</update_rate>
           <ray>
@@ -95,5 +95,5 @@
         <sensor type="ray" name="${name}-VLP16">
           <pose>0 0 0 0 0 0</pose>
-          <visualize>false</visualize>
+          <visualize>true</visualize>
           <update_rate>${hz}</update_rate>
           <ray>

File: src/velodyne_description/urdf/VLP-32C.urdf.xacro (robot description, xacro)
@@ -55,5 +55,5 @@
         <sensor type="gpu_ray" name="${name}-VLP32C">
           <pose>0 0 0 0 0 0</pose>
-          <visualize>false</visualize>
+          <visualize>true</visualize>
           <update_rate>${hz}</update_rate>
           <ray>
@@ -109,5 +109,5 @@
         <sensor type="ray" name="${name}-VLP32C">
           <pose>0 0 0 0 0 0</pose>
-          <visualize>false</visualize>
+          <visualize>true</visualize>
           <update_rate>${hz}</update_rate>
           <ray>

File: src/velodyne_description/urdf/example.urdf.xacro (robot description, xacro)
@@ -30,13 +30,13 @@
     </inertial>
   </link>
-  <xacro:include filename="$(find velodyne_description)/urdf/VLP-16.urdf.xacro"/>
+  <xacro:include filename="VLP-16.urdf.xacro"/>
   <VLP-16 parent="base_link" name="velodyne" topic="/velodyne_points" hz="10" samples="440" gpu="${gpu}">
     <origin xyz="0 0 0.4" rpy="0 0 0" />
   </VLP-16>
-  <xacro:include filename="$(find velodyne_description)/urdf/HDL-32E.urdf.xacro"/>
-   <HDL-32E parent="base_link" name="velodyne2" topic="/velodyne_points2" hz="10" samples="220" gpu="${gpu}">
+  <xacro:include filename="HDL-32E.urdf.xacro"/>
+  <HDL-32E parent="base_link" name="velodyne2" topic="/velodyne_points2" hz="10" samples="220" gpu="${gpu}">
     <origin xyz="0 0 0.6" rpy="0 0 0" />
   </HDL-32E>
-  <xacro:include filename="$(find velodyne_description)/urdf/VLP-32C.urdf.xacro"/>
+  <xacro:include filename="VLP-32C.urdf.xacro"/>
   <VLP-32C parent="base_link" name="velodyne3" topic="/velodyne_points3" hz="10" samples="1200" gpu="${gpu}">
     <origin xyz="0 0 0.8" rpy="0 0 0" />
